Commit message: modified urdf

File: sawyer/sawyer.urdf (robot description, URDF)
Before this commit: robot sawyer, 21 links, 20 joints
Links:
- added link controller_box; collision box size=0.22 0.4 0.53
- added link pedestal, mass 60.86397744; collision cylinder length=0.62 radius=0.18; visual mesh filename=meshes/sawyer_pv/pedestal.STL
- added link pedestal_feet; collision box size=0.77 0.7 0.31
Joints:
- added joint controller_box_fixed: type fixed, parent base, child controller_box, origin xyz=0.0 0.0 0.0 rpy=0 0 0
- added joint pedestal_feet_fixed: type fixed, parent base, child pedestal_feet, origin xyz=0.0 0.0 0.0 rpy=0 0 0
- added joint pedestal_fixed: type fixed, parent base, child pedestal, origin xyz=0.0 0.0 0.0 rpy=0 0 0

Commit message: modified sawyer.urdf

File: sawyer/sawyer.urdf (robot description, URDF)
Before this commit: robot sawyer, 24 links, 23 joints
Joints:
- joint sawyer_right_hand: origin xyz=0 0 0.0245 rpy=0 0 1.570796 -> xyz=0 0 0.024 rpy=0 0 0
