Commit message: modified urdfg

File: panda/panda.urdf (robot description, URDF)
Before this commit: robot panda, 15 links, 14 joints
Links:
- removed link controller_box
- removed link pedestal
- removed link pedestal_feet
- added link panda_controller_box; collision box size=0.22 0.4 0.53
- added link panda_pedestal, mass 60.86397744; collision cylinder length=0.62 radius=0.18; visual mesh filename=meshes/sawyer_pv/pedestal.STL
- added link panda_pedestal_feet; collision box size=0.77 0.7 0.31
Joints:
- removed joint controller_box_fixed
- removed joint pedestal_feet_fixed
- removed joint pedestal_fixed
- added joint panda_controller_box_fixed: type fixed, parent base, child controller_box, origin xyz=0.0 0.0 0.0 rpy=0 0 0
- added joint panda_pedestal_feet_fixed: type fixed, parent pedestal_feet, child panda_link0, origin xyz=0.0 0.0 0.0 rpy=0 0 0
- added joint panda_pedestal_fixed: type fixed, parent panda_pedestal, child panda_link0, origin xyz=0.0 0.0 0.0 rpy=0 0 0

File: sawyer/sawyer.urdf (robot description, URDF)
Before this commit: robot sawyer, 24 links, 23 joints
Links:
- removed link base
- removed link controller_box
- removed link head
- removed link head_camera
- removed link pedestal
- removed link pedestal_feet
- removed link right_arm_base_link
- removed link right_arm_itb
- removed link right_hand
- removed link right_hand_camera
- removed link right_l0
- removed link right_l1
- removed link right_l1_2
- removed link right_l2
- removed link right_l2_2
- removed link right_l3
- removed link right_l4
- removed link right_l4_2
- removed link right_l5
- removed link right_l6
- removed link right_torso_itb
- removed link right_wrist
- removed link screen
- removed link torso
- added link sawyer_base
- added link sawyer_controller_box; collision box size=0.22 0.4 0.53
- added link sawyer_head, mass 1.5795; collision sphere radius=0.18; visual mesh filename=meshes/sawyer_pv/head.STL
- added link sawyer_head_camera
- added link sawyer_pedestal, mass 60.86397744; collision cylinder length=0.62 radius=0.18; visual mesh filename=meshes/sawyer_pv/pedestal.STL
- added link sawyer_pedestal_feet; collision box size=0.77 0.7 0.31
- added link sawyer_right_arm_base_link, mass 2.0687; collision cylinder length=0.24 radius=0.08; visual mesh filename=meshes/sawyer_pv/base.STL
- added link sawyer_right_arm_itb
- added link sawyer_right_hand; collision cylinder length=0.03 radius=0.035
- added link sawyer_right_hand_camera
- added link sawyer_right_l0, mass 5.3213; collision sphere radius=0.07; visual mesh filename=meshes/sawyer_mp3/l0.STL
- added link sawyer_right_l1, mass 4.505; collision sphere radius=0.07; visual mesh filename=meshes/sawyer_mp3/l1.STL
- added link sawyer_right_l1_2; collision cylinder length=0.14 radius=0.07
- added link sawyer_right_l2, mass 1.745; collision cylinder length=0.34 radius=0.06; visual mesh filename=meshes/sawyer_pv/l2.STL
- added link sawyer_right_l2_2; collision sphere radius=0.06
- added link sawyer_right_l3, mass 2.5097; collision sphere radius=0.06; visual mesh filename=meshes/sawyer_pv/l3.STL
- added link sawyer_right_l4, mass 1.1136; collision cylinder length=0.30 radius=0.045; visual mesh filename=meshes/sawyer_pv/l4.STL
- added link sawyer_right_l4_2; collision sphere radius=0.06
- added link sawyer_right_l5, mass 1.5625; collision sphere radius=0.06; visual mesh filename=meshes/sawyer_pv/l5.STL
- added link sawyer_right_l6, mass 0.3292; collision cylinder length=0.05 radius=0.055; visual mesh filename=meshes/sawyer_mp1/l6.STL
- added link sawyer_right_torso_itb
- added link sawyer_right_wrist
- added link sawyer_screen; collision sphere radius=0.001; visual box size=0.24 0.14 0.002
- added link sawyer_torso; visual box size=0.001 0.001 0.001
Joints:
- removed joint controller_box_fixed
- removed joint display_joint
- removed joint head_camera
- removed joint head_pan
- removed joint pedestal_feet_fixed
- removed joint pedestal_fixed
- removed joint right_arm_itb
- removed joint right_arm_mount
- removed joint right_hand
- removed joint right_hand_camera
- removed joint right_j0
- removed joint right_j1
- removed joint right_j1_2
- removed joint right_j2
- removed joint right_j2_2
- removed joint right_j3
- removed joint right_j4
- removed joint right_j4_2
- removed joint right_j5
- removed joint right_j6
- removed joint right_torso_itb
- removed joint right_wrist
- removed joint torso_t0
- added joint sawyer_controller_box_fixed: type fixed, parent sawyer_base, child sawyer_controller_box, origin xyz=0.0 0.0 0.0 rpy=0 0 0
- added joint sawyer_display_joint: type fixed, parent sawyer_head, child sawyer_screen, origin xyz=0.03 0.0 0.105 rpy=1.57079632679 0 1.57079632679
- added joint sawyer_head_camera: type fixed, parent sawyer_head, child sawyer_head_camera, origin xyz=0.0228027 0 0.216572 rpy=-2.1293 0 -1.57079632679, axis 0 0 0
- added joint sawyer_head_pan: type revolute, parent sawyer_right_l0, child sawyer_head, origin xyz=0 0 0.2965 rpy=0 0 0, axis 0 0 1, limit lower=-5.0952 upper=0.9064 effort=8 velocity=1.8
- added joint sawyer_pedestal_feet_fixed: type fixed, parent sawyer_base, child sawyer_pedestal_feet, origin xyz=0.0 0.0 0.0 rpy=0 0 0
- added joint sawyer_pedestal_fixed: type fixed, parent sawyer_base, child sawyer_pedestal, origin xyz=0.0 0.0 0.0 rpy=0 0 0
- added joint sawyer_right_arm_itb: type fixed, parent sawyer_right_l4, child sawyer_right_arm_itb, origin xyz=-.055 0 .075 rpy=0 -1.57079632679 0, axis 0 0 1
- added joint sawyer_right_arm_mount: type fixed, parent sawyer_base, child sawyer_right_arm_base_link, origin xyz=0.0 0.0 0.0 rpy=0 0 0
- added joint sawyer_right_hand: type fixed, parent sawyer_right_l6, child sawyer_right_hand, origin xyz=0 0 0.0245 rpy=0 0 1.570796, axis 0 0 1
- added joint sawyer_right_hand_camera: type fixed, parent sawyer_right_l5, child sawyer_right_hand_camera, origin xyz=0.039552 -0.033 0.0695 rpy=0 1.57079632679 0, axis 0 0 0
- added joint sawyer_right_j0: type revolute, parent sawyer_right_arm_base_link, child sawyer_right_l0, origin xyz=0 0 0.08 rpy=0 0 0, axis 0 0 1, limit lower=-3.0503 upper=3.0503 effort=80.0 velocity=1.74
- added joint sawyer_right_j1: type revolute, parent sawyer_right_l0, child sawyer_right_l1, origin xyz=0.081 0.05 0.237 rpy=-1.57079632679 1.57079632679 0, axis 0 0 1, limit lower=-3.8095 upper=2.2736 effort=80.0 velocity=1.328
- added joint sawyer_right_j1_2: type fixed, parent sawyer_right_l1, child sawyer_right_l1_2, origin xyz=0 0 0 rpy=0 0 0, axis 0 0 1
- added joint sawyer_right_j2: type revolute, parent sawyer_right_l1, child sawyer_right_l2, origin xyz=0 -0.14 0.1425 rpy=1.57079632679 0 0, axis 0 0 1, limit lower=-3.0426 upper=3.0426 effort=40.0 velocity=1.957
- added joint sawyer_right_j2_2: type fixed, parent sawyer_right_l2, child sawyer_right_l2_2, origin xyz=0 0 0 rpy=0 0 0, axis 0 0 1
- added joint sawyer_right_j3: type revolute, parent sawyer_right_l2, child sawyer_right_l3, origin xyz=0 -0.042 0.26 rpy=-1.57079632679 0 0, axis 0 0 1, limit lower=-3.0439 upper=3.0439 effort=40.0 velocity=1.957
- added joint sawyer_right_j4: type revolute, parent sawyer_right_l3, child sawyer_right_l4, origin xyz=0 -0.125 -0.1265 rpy=1.57079632679 0 0, axis 0 0 1, limit lower=-2.9761 upper=2.9761 effort=9.0 velocity=3.485
- added joint sawyer_right_j4_2: type fixed, parent sawyer_right_l4, child sawyer_right_l4_2, origin xyz=0 0 0 rpy=0 0 0, axis 0 0 1
- added joint sawyer_right_j5: type revolute, parent sawyer_right_l4, child sawyer_right_l5, origin xyz=0 0.031 0.275 rpy=-1.57079632679 0 0, axis 0 0 1, limit lower=-2.9761 upper=2.9761 effort=9.0 velocity=3.485
- added joint sawyer_right_j6: type revolute, parent sawyer_right_l5, child sawyer_right_l6, origin xyz=0 -0.11 0.1053 rpy=-1.57079632679 -0.17453 3.1416, axis 0 0 1
- added joint sawyer_right_torso_itb: type fixed, parent sawyer_right_l0, child sawyer_right_torso_itb, origin xyz=-.055 0 .22 rpy=0 -1.57079632679 0, axis 0 0 1
- added joint sawyer_right_wrist: type fixed, parent sawyer_right_l5, child sawyer_right_wrist, origin xyz=0 0 0.10541 rpy=1.57079632679 0 0, axis 0 0 0
- added joint sawyer_torso_t0: type fixed, parent sawyer_base, child sawyer_torso, origin xyz=0 0 0 rpy=0 0 0

Commit message: modified panda urdf

File: panda/panda.urdf (robot description, URDF)
Before this commit: robot panda, 15 links, 14 joints
Joints:
- joint panda_joint7: origin xyz=0.088 0 0 rpy=1.57079632679 0 0 -> xyz=0.088 0 0 rpy=1.57079632679 0 0.7854

Commit message: modified panda urdf

File: panda/panda.urdf (robot description, URDF)
Before this commit: robot panda, 15 links, 14 joints
Links:
- removed link panda_hand
- removed link panda_link8
- added link panda_finger_joint1_tip; collision mesh filename=meshes/collision/finger.stl
- added link panda_finger_joint2_tip; collision mesh filename=meshes/collision/finger.stl
- added link panda_right_gripper; collision mesh filename=meshes/collision/hand.stl; visual mesh filename=meshes/collision/hand.stl
- added link panda_right_hand
Joints:
- removed joint panda_hand_joint
- removed joint panda_joint8
- added joint anda_finger_joint2_tip_fixed: type fixed, parent panda_rightfinger, child panda_finger_joint2_tip, origin xyz=0 -0.0085 0.056 rpy=0 0 0
- added joint panda_finger_joint1_tip_fixed: type fixed, parent panda_leftfinger, child panda_finger_joint1_tip, origin xyz=0 0.0085 0.056 rpy=0 0 0
- added joint panda_joint9: type fixed, parent panda_right_hand, child panda_right_gripper, origin xyz=0 0 0 rpy=0 0 -1.5707963, axis 0 0 0
- added joint panda_right_hand_fixed: type fixed, parent panda_link7, child panda_right_hand, origin xyz=0 0 0.1065 rpy=0 0 -0.7858908
- joint panda_finger_joint1: origin xyz=0 0 0.0584 rpy=0 0 0 -> xyz=0 0 0.0524 rpy=0 0 0; parent panda_hand -> panda_right_gripper
- joint panda_finger_joint2: mimic joint=panda_finger_joint1 -> (none); origin xyz=0 0 0.0584 rpy=0 0 0 -> xyz=0 0 0.0524 rpy=0 0 0; parent panda_hand -> panda_right_gripper
- joint panda_joint7: origin xyz=0.088 0 0 rpy=1.57079632679 0 0.7854 -> xyz=0.088 0 0 rpy=1.57079632679 0.7854 0

Commit message: modified panda.urdf

File: panda/panda.urdf (robot description, URDF)
Before this commit: robot panda, 17 links, 16 joints
Joints:
- joint panda_joint7: origin xyz=0.088 0 0 rpy=1.57079632679 0.7854 0 -> xyz=0.088 0 0 rpy=1.57079632679 0 0

Commit message: modified panda.urdf

File: panda/panda.urdf (robot description, URDF)
Before this commit: robot panda, 17 links, 16 joints
Links:
- removed link panda_leftfinger
- removed link panda_right_gripper
- removed link panda_rightfinger
- added link gripper; collision mesh filename=meshes/collision/hand.stl; visual mesh filename=meshes/collision/hand.stl
- added link leftfinger; collision mesh filename=meshes/collision/finger.stl; visual mesh filename=meshes/collision/finger.stl
- added link rightfinger; collision mesh filename=meshes/collision/finger.stl; visual mesh filename=meshes/collision/finger.stl
Joints:
- joint anda_finger_joint2_tip_fixed: parent panda_rightfinger -> rightfinger
- joint panda_finger_joint1: child panda_leftfinger -> leftfinger; parent panda_right_gripper -> gripper
- joint panda_finger_joint2: child panda_rightfinger -> rightfinger; parent panda_right_gripper -> gripper
- joint panda_right_gripper_fixed: child panda_right_gripper -> gripper; origin xyz=0 0 0 rpy=0 0 -1.5707963 -> xyz=0 0 0 rpy=0 0 -3.1415926

Commit message: modified panda.urdf

File: panda/panda.urdf (robot description, URDF)
Before this commit: robot panda, 17 links, 16 joints
Links:
- removed link gripper
- removed link panda_finger_joint1_tip
- removed link panda_finger_joint2_tip
- added link right_gripper; collision mesh filename=meshes/collision/hand.stl; visual mesh filename=meshes/collision/hand.stl
Joints:
- removed joint anda_finger_joint2_tip_fixed
- removed joint panda_finger_joint1_tip_fixed
- removed joint panda_right_gripper_fixed
- added joint panda_right_right_gripper_fixed: type fixed, parent panda_right_hand, child right_gripper, origin xyz=0 0 0 rpy=0 0 -1.5707963, axis 0 0 0
- joint panda_finger_joint1: origin xyz=0 0 0.0524 rpy=0 0 0 -> xyz=0 0 0.0524 rpy=0 0 1.5707963; parent gripper -> right_gripper
- joint panda_finger_joint2: axis 0 -1 0 -> 0 1 0; origin xyz=0 0 0.0524 rpy=0 0 0 -> xyz=0 0 0.0524 rpy=0 0 1.5707963; parent gripper -> right_gripper

Commit message: modifiled panda.urdf

File: panda/panda.urdf (robot description, URDF)
Before this commit: robot panda, 15 links, 14 joints
Links:
- link leftfinger: geometry collision mesh filename=meshes/collision/finger.stl; visual mesh filename=meshes/visual/finger.stl
- link panda_link_0: geometry collision mesh filename=meshes/collision/link0.stl; visual mesh filename=meshes/visual/link0.stl
- link panda_link_1: geometry collision mesh filename=meshes/collision/link1.stl; visual mesh filename=meshes/visual/link1.stl
- link panda_link_2: geometry collision mesh filename=meshes/collision/link2.stl; visual mesh filename=meshes/visual/link2.stl
- link panda_link_3: geometry collision mesh filename=meshes/collision/link3.stl; visual mesh filename=meshes/visual/link3.stl
- link panda_link_4: geometry collision mesh filename=meshes/collision/link4.stl; visual mesh filename=meshes/visual/link4.stl
- link panda_link_5: geometry collision mesh filename=meshes/collision/link5.stl; visual mesh filename=meshes/visual/link5.stl
- link panda_link_6: geometry collision mesh filename=meshes/collision/link6.stl; visual mesh filename=meshes/visual/link6.stl
- link panda_link_7: geometry collision mesh filename=meshes/collision/link7.stl; visual mesh filename=meshes/visual/link7.stl
- link panda_pedestal: geometry collision mesh filename=meshes/panda_pedestal/pedestal.STL; visual mesh filename=meshes/panda_pedestal/pedestal.STL
- link right_gripper: geometry collision mesh filename=meshes/collision/hand.stl; visual mesh filename=meshes/visual/hand.stl
- link rightfinger: geometry collision mesh filename=meshes/collision/finger.stl; visual mesh filename=meshes/visual/finger.stl

Commit message: modified panda.urdf

File: panda/panda.urdf (robot description, URDF)
Before this commit: robot panda, 15 links, 14 joints
Joints:
- joint panda_finger_joint1: origin xyz=0 0 0.0524 rpy=0 0 1.5707963 -> xyz=-0.04 0 0.0524 rpy=0 0 1.5707963
- joint panda_finger_joint2: origin xyz=0 0 0.0524 rpy=0 0 1.5707963 -> xyz=0.04 0 0.0524 rpy=0 0 1.5707963

Commit message: modified panda.urdf

File: panda/panda.urdf (robot description, URDF)
Before this commit: robot panda, 15 links, 14 joints
Links:
- added link tcp
Joints:
- added joint panda_eef_fixed: type fixed, parent panda_right_hand, child tcp, origin xyz=0 0 0.097 rpy=0 0 0

Commit message: modified panda.urdf

File: panda/panda.urdf (robot description, URDF)
Before this commit: robot panda, 16 links, 15 joints
Links:
- link panda_pedestal: geometry collision cylinder length=0.62 radius=0.18; visual mesh filename=meshes/panda_pedestal/pedestal.STL
Joints:
- joint panda_controller_box_fixed: child controller_box -> panda_controller_box; parent base -> panda_link_0
- joint panda_pedestal_feet_fixed: child panda_link_0 -> panda_pedestal_feet; parent pedestal_feet -> panda_link_0
- joint panda_pedestal_fixed: child panda_link_0 -> panda_pedestal; parent panda_pedestal -> panda_link_0
