Commit message: modified urdf

File: iiwa14/iiwa14.urdf (robot description, URDF)
Before this commit: robot iiwa14, 9 links, 8 joints
Links:
- added link controller_box; collision box size=0.22 0.4 0.53
- added link panda_link1; collision mesh filename=meshes/iiwa14/collision/link1.stl; visual mesh filename=meshes/iiwa14/collision/link1.stl
- added link pedestal, mass 60.86397744; collision cylinder length=0.62 radius=0.18; visual mesh filename=meshes/iiwa14/sawyer_pv/pedestal.STL
- added link pedestal_feet; collision box size=0.77 0.7 0.31
Joints:
- added joint controller_box_fixed: type fixed, parent base, child controller_box, origin xyz=0.0 0.0 0.0 rpy=0 0 0
- added joint pedestal_feet_fixed: type fixed, parent pedestal_feet, child iiwa_link_0, origin xyz=0.0 0.0 0.0 rpy=0 0 0
- added joint pedestal_fixed: type fixed, parent pedestal, child iiwa_link_0, origin xyz=0.0 0.0 0.0 rpy=0 0 0

File: panda/panda.urdf (robot description, URDF)
Before this commit: robot panda, 12 links, 11 joints
Links:
- added link controller_box; collision box size=0.22 0.4 0.53
- added link pedestal, mass 60.86397744; collision cylinder length=0.62 radius=0.18; visual mesh filename=meshes/sawyer_pv/pedestal.STL
- added link pedestal_feet; collision box size=0.77 0.7 0.31
Joints:
- added joint controller_box_fixed: type fixed, parent base, child controller_box, origin xyz=0.0 0.0 0.0 rpy=0 0 0
- added joint pedestal_feet_fixed: type fixed, parent pedestal_feet, child panda_link0, origin xyz=0.0 0.0 0.0 rpy=0 0 0
- added joint pedestal_fixed: type fixed, parent pedestal, child panda_link0, origin xyz=0.0 0.0 0.0 rpy=0 0 0

Commit message: modified iiwa14.urdf

File: iiwa14/iiwa14.urdf (robot description, URDF)
Before this commit: robot iiwa14, 13 links, 11 joints
Links:
- removed link panda_link1

Commit message: modified iiwa14.urdf

File: iiwa14/iiwa14.urdf (robot description, URDF)
Before this commit: robot iiwa14, 12 links, 11 joints
Links:
- removed link iiwa_link_0
- removed link iiwa_link_1
- removed link iiwa_link_2
- removed link iiwa_link_3
- removed link iiwa_link_4
- removed link iiwa_link_5
- removed link iiwa_link_6
- removed link iiwa_link_7
- removed link iiwa_link_ee
- added link iiwa14_link_0, mass 5; collision mesh filename=meshes/iiwa14/collision/link_0.stl; visual mesh filename=meshes/iiwa14/visual/link_0.stl
- added link iiwa14_link_1, mass 4; collision mesh filename=meshes/iiwa14/collision/link_1.stl; visual mesh filename=meshes/iiwa14/visual/link_1.stl
- added link iiwa14_link_2, mass 4; collision mesh filename=meshes/iiwa14/collision/link_2.stl; visual mesh filename=meshes/iiwa14/visual/link_2.stl
- added link iiwa14_link_3, mass 3; collision mesh filename=meshes/iiwa14/collision/link_3.stl; visual mesh filename=meshes/iiwa14/visual/link_3.stl
- added link iiwa14_link_4, mass 2.7; collision mesh filename=meshes/iiwa14/collision/link_4.stl; visual mesh filename=meshes/iiwa14/visual/link_4.stl
- added link iiwa14_link_5, mass 1.7; collision mesh filename=meshes/iiwa14/collision/link_5.stl; visual mesh filename=meshes/iiwa14/visual/link_5.stl
- added link iiwa14_link_6, mass 1.8; collision mesh filename=meshes/iiwa14/collision/link_6.stl; visual mesh filename=meshes/iiwa14/visual/link_6.stl
- added link iiwa14_link_7, mass 0.3; collision mesh filename=meshes/iiwa14/collision/link_7.stl; visual mesh filename=meshes/iiwa14/visual/link_7.stl
- added link iiwa14_link_ee, mass 0
Joints:
- removed joint iiwa_joint_1
- removed joint iiwa_joint_2
- removed joint iiwa_joint_3
- removed joint iiwa_joint_4
- removed joint iiwa_joint_5
- removed joint iiwa_joint_6
- removed joint iiwa_joint_7
- removed joint iiwa_joint_ee
- added joint iiwa14_joint_1: type revolute, parent iiwa14_link_0, child iiwa14_link_1, origin xyz=0 0 0.1575 rpy=0 0 0, axis 0 0 1, limit lower=-2.96705972839 upper=2.96705972839 effort=300 velocity=10
- added joint iiwa14_joint_2: type revolute, parent iiwa14_link_1, child iiwa14_link_2, origin xyz=0 0 0.2025 rpy=1.57079632679   0 3.14159265359, axis 0 0 1, limit lower=-2.09439510239 upper=2.09439510239 effort=300 velocity=10
- added joint iiwa14_joint_3: type revolute, parent iiwa14_link_2, child iiwa14_link_3, origin xyz=0 0.2045 0 rpy=1.57079632679 0 3.14159265359, axis 0 0 1, limit lower=-2.96705972839 upper=2.96705972839 effort=300 velocity=10
- added joint iiwa14_joint_4: type revolute, parent iiwa14_link_3, child iiwa14_link_4, origin xyz=0 0 0.2155 rpy=1.57079632679 0 0, axis 0 0 1, limit lower=-2.09439510239 upper=2.09439510239 effort=300 velocity=10
- added joint iiwa14_joint_5: type revolute, parent iiwa14_link_4, child iiwa14_link_5, origin xyz=0 0.1845 0 rpy=-1.57079632679 3.14159265359 0, axis 0 0 1, limit lower=-2.96705972839 upper=2.96705972839 effort=300 velocity=10
- added joint iiwa14_joint_6: type revolute, parent iiwa14_link_5, child iiwa14_link_6, origin xyz=0 0 0.2155 rpy=1.57079632679 0 0, axis 0 0 1, limit lower=-2.09439510239 upper=2.09439510239 effort=300 velocity=10
- added joint iiwa14_joint_7: type revolute, parent iiwa14_link_6, child iiwa14_link_7, origin xyz=0 0.081 0 rpy=-1.57079632679 3.14159265359 0, axis 0 0 1, limit lower=-3.05432619099 upper=3.05432619099 effort=300 velocity=10
- added joint iiwa14_joint_ee: type fixed, parent iiwa14_link_7, child iiwa14_link_ee, origin xyz=0 0 0.045 rpy=0 0 0
- joint pedestal_feet_fixed: child iiwa_link_0 -> iiwa14_link_0
- joint pedestal_fixed: child iiwa_link_0 -> iiwa14_link_0

Commit message: modified urdf

File: iiwa14/iiwa14.urdf (robot description, URDF)
Before this commit: robot iiwa14, 12 links, 11 joints
Links:
- added link panda_link1; collision mesh filename=meshes/iiwa14/collision/link1.stl; visual mesh filename=meshes/iiwa14/collision/link1.stl
- link pedestal: geometry collision cylinder length=0.62 radius=0.18; visual mesh filename=meshes/iiwa14/iiwa14_pedestal/pedestal.STL

File: iiwa7/iiwa7.urdf (robot description, URDF)
Before this commit: robot iiwa7, 12 links, 11 joints
Links:
- link pedestal: geometry collision cylinder length=0.62 radius=0.18; visual mesh filename=meshes/iiwa7/iiwa7_pedestal/pedestal.STL

File: panda/panda.urdf (robot description, URDF)
Before this commit: robot panda, 15 links, 14 joints
Links:
- link panda_pedestal: geometry collision cylinder length=0.62 radius=0.18; visual mesh filename=meshes/panda_pedestal/pedestal.STL

Commit message: modified eef name

File: iiwa14/iiwa14.urdf (robot description, URDF)
Before this commit: robot iiwa14, 13 links, 11 joints
Links:
- removed link iiwa14_link_ee
- added link iiwa14_right_hand, mass 0
Joints:
- removed joint iiwa14_joint_ee
- added joint iiwa14_joint_right_hand_fixed: type fixed, parent iiwa14_link_7, child iiwa14_right_hand, origin xyz=0 0 0.045 rpy=0 0 0

File: iiwa7/iiwa7.urdf (robot description, URDF)
Before this commit: robot iiwa7, 12 links, 11 joints
Links:
- removed link iiwa7_link_ee
- added link iiwa7_right_hand, mass 0
Joints:
- removed joint iiwa7_joint_ee
- added joint iiwa7_right_hand_fixed: type fixed, parent iiwa7_link_7, child iiwa7_right_hand, origin xyz=0 0 0.044 rpy=0 0 0

File: panda/panda.urdf (robot description, URDF)
Before this commit: robot panda, 17 links, 16 joints
Joints:
- removed joint panda_joint9
- added joint panda_right_gripper_fixed: type fixed, parent panda_right_hand, child panda_right_gripper, origin xyz=0 0 0 rpy=0 0 -1.5707963, axis 0 0 0

Commit message: modified link names

File: iiwa14/iiwa14.urdf (robot description, URDF)
Before this commit: robot iiwa14, 13 links, 11 joints
Links:
- removed link panda_link1

File: panda/panda.urdf (robot description, URDF)
Before this commit: robot panda, 15 links, 14 joints
Links:
- removed link panda_link0
- removed link panda_link1
- removed link panda_link2
- removed link panda_link3
- removed link panda_link4
- removed link panda_link5
- removed link panda_link6
- removed link panda_link7
- added link panda_link_0; collision mesh filename=meshes/collision/link0.stl; visual mesh filename=meshes/collision/link0.stl
- added link panda_link_1; collision mesh filename=meshes/collision/link1.stl; visual mesh filename=meshes/collision/link1.stl
- added link panda_link_2; collision mesh filename=meshes/collision/link2.stl; visual mesh filename=meshes/collision/link2.stl
- added link panda_link_3; collision mesh filename=meshes/collision/link3.stl; visual mesh filename=meshes/collision/link3.stl
- added link panda_link_4; collision mesh filename=meshes/collision/link4.stl; visual mesh filename=meshes/collision/link4.stl
- added link panda_link_5; collision mesh filename=meshes/collision/link5.stl; visual mesh filename=meshes/collision/link5.stl
- added link panda_link_6; collision mesh filename=meshes/collision/link6.stl; visual mesh filename=meshes/collision/link6.stl
- added link panda_link_7; collision mesh filename=meshes/collision/link7.stl; visual mesh filename=meshes/collision/link7.stl
Joints:
- joint panda_joint1: child panda_link1 -> panda_link_1; parent panda_link0 -> panda_link_0
- joint panda_joint2: child panda_link2 -> panda_link_2; parent panda_link1 -> panda_link_1
- joint panda_joint3: child panda_link3 -> panda_link_3; parent panda_link2 -> panda_link_2
- joint panda_joint4: child panda_link4 -> panda_link_4; parent panda_link3 -> panda_link_3
- joint panda_joint5: child panda_link5 -> panda_link_5; parent panda_link4 -> panda_link_4
- joint panda_joint6: child panda_link6 -> panda_link_6; parent panda_link5 -> panda_link_5
- joint panda_joint7: child panda_link7 -> panda_link_7; parent panda_link6 -> panda_link_6
- joint panda_pedestal_feet_fixed: child panda_link0 -> panda_link_0
- joint panda_pedestal_fixed: child panda_link0 -> panda_link_0
- joint panda_right_hand_fixed: parent panda_link7 -> panda_link_7

File: sawyer/sawyer.urdf (robot description, URDF)
Before this commit: robot sawyer, 24 links, 23 joints
Links:
- removed link sawyer_right_l0
- removed link sawyer_right_l1
- removed link sawyer_right_l1_2
- removed link sawyer_right_l2
- removed link sawyer_right_l2_2
- removed link sawyer_right_l3
- removed link sawyer_right_l4
- removed link sawyer_right_l4_2
- removed link sawyer_right_l5
- removed link sawyer_right_l6
- added link sawyer_link_0, mass 5.3213; collision sphere radius=0.07; visual mesh filename=meshes/sawyer_mp3/l0.STL
- added link sawyer_link_1, mass 4.505; collision sphere radius=0.07; visual mesh filename=meshes/sawyer_mp3/l1.STL
- added link sawyer_link_1_2; collision cylinder length=0.14 radius=0.07
- added link sawyer_link_2, mass 1.745; collision cylinder length=0.34 radius=0.06; visual mesh filename=meshes/sawyer_pv/l2.STL
- added link sawyer_link_2_2; collision sphere radius=0.06
- added link sawyer_link_3, mass 2.5097; collision sphere radius=0.06; visual mesh filename=meshes/sawyer_pv/l3.STL
- added link sawyer_link_4, mass 1.1136; collision cylinder length=0.30 radius=0.045; visual mesh filename=meshes/sawyer_pv/l4.STL
- added link sawyer_link_4_2; collision sphere radius=0.06
- added link sawyer_link_5, mass 1.5625; collision sphere radius=0.06; visual mesh filename=meshes/sawyer_pv/l5.STL
- added link sawyer_link_6, mass 0.3292; collision cylinder length=0.05 radius=0.055; visual mesh filename=meshes/sawyer_mp1/l6.STL
Joints:
- joint sawyer_head_pan: parent sawyer_right_l0 -> sawyer_link_0
- joint sawyer_right_arm_itb: parent sawyer_right_l4 -> sawyer_link_4
- joint sawyer_right_hand: parent sawyer_right_l6 -> sawyer_link_6
- joint sawyer_right_hand_camera: parent sawyer_right_l5 -> sawyer_link_5
- joint sawyer_right_j0: child sawyer_right_l0 -> sawyer_link_0
- joint sawyer_right_j1: child sawyer_right_l1 -> sawyer_link_1; parent sawyer_right_l0 -> sawyer_link_0
- joint sawyer_right_j1_2: child sawyer_right_l1_2 -> sawyer_link_1_2; parent sawyer_right_l1 -> sawyer_link_1
- joint sawyer_right_j2: child sawyer_right_l2 -> sawyer_link_2; parent sawyer_right_l1 -> sawyer_link_1
- joint sawyer_right_j2_2: child sawyer_right_l2_2 -> sawyer_link_2_2; parent sawyer_right_l2 -> sawyer_link_2
- joint sawyer_right_j3: child sawyer_right_l3 -> sawyer_link_3; parent sawyer_right_l2 -> sawyer_link_2
- joint sawyer_right_j4: child sawyer_right_l4 -> sawyer_link_4; parent sawyer_right_l3 -> sawyer_link_3
- joint sawyer_right_j4_2: child sawyer_right_l4_2 -> sawyer_link_4_2; parent sawyer_right_l4 -> sawyer_link_4
- joint sawyer_right_j5: child sawyer_right_l5 -> sawyer_link_5; parent sawyer_right_l4 -> sawyer_link_4
- joint sawyer_right_j6: child sawyer_right_l6 -> sawyer_link_6; parent sawyer_right_l5 -> sawyer_link_5
- joint sawyer_right_torso_itb: parent sawyer_right_l0 -> sawyer_link_0
- joint sawyer_right_wrist: parent sawyer_right_l5 -> sawyer_link_5

Commit message: modified iiwa14 iiwa7 ur5e urdf

File: iiwa14/iiwa14.urdf (robot description, URDF)
Before this commit: robot iiwa14, 12 links, 11 joints
Links:
- removed link controller_box
- removed link pedestal
- removed link pedestal_feet
- added link iiwa14_controller_box; collision box size=0.22 0.4 0.53
- added link iiwa14_pedestal, mass 60.86397744; collision cylinder length=0.62 radius=0.18; visual mesh filename=meshes/iiwa14_pedestal/pedestal.STL
- added link iiwa14_pedestal_feet; collision box size=0.77 0.7 0.31
- link iiwa14_link_0: geometry collision mesh filename=meshes/collision/link_0.stl; visual mesh filename=meshes/visual/link_0.stl
- link iiwa14_link_1: geometry collision mesh filename=meshes/collision/link_1.stl; visual mesh filename=meshes/visual/link_1.stl
- link iiwa14_link_2: geometry collision mesh filename=meshes/collision/link_2.stl; visual mesh filename=meshes/visual/link_2.stl
- link iiwa14_link_3: geometry collision mesh filename=meshes/collision/link_3.stl; visual mesh filename=meshes/visual/link_3.stl
- link iiwa14_link_4: geometry collision mesh filename=meshes/collision/link_4.stl; visual mesh filename=meshes/visual/link_4.stl
- link iiwa14_link_5: geometry collision mesh filename=meshes/collision/link_5.stl; visual mesh filename=meshes/visual/link_5.stl
- link iiwa14_link_6: geometry collision mesh filename=meshes/collision/link_6.stl; visual mesh filename=meshes/visual/link_6.stl
- link iiwa14_link_7: geometry collision mesh filename=meshes/collision/link_7.stl; visual mesh filename=meshes/visual/link_7.stl
Joints:
- removed joint controller_box_fixed
- removed joint pedestal_feet_fixed
- removed joint pedestal_fixed
- added joint iiwa14_controller_box_fixed: type fixed, parent iiwa14_link_0, child iiwa14_controller_box, origin xyz=0.0 0.0 0.0 rpy=0 0 0
- added joint iiwa14_pedestal_feet_fixed: type fixed, parent iiwa14_link_0, child iiwa14_pedestal_feet, origin xyz=0.0 0.0 0.0 rpy=0 0 0
- added joint iiwa14_pedestal_fixed: type fixed, parent iiwa14_link_0, child iiwa14_pedestal, origin xyz=0.0 0.0 0.0 rpy=0 0 0

File: iiwa7/iiwa7.urdf (robot description, URDF)
Before this commit: robot iiwa7, 12 links, 11 joints
Links:
- removed link controller_box
- removed link pedestal
- removed link pedestal_feet
- added link iiwa7_controller_box; collision box size=0.22 0.4 0.53
- added link iiwa7_pedestal, mass 60.86397744; collision cylinder length=0.62 radius=0.18; visual mesh filename=meshes/iiwa7_pedestal/pedestal.STL
- added link iiwa7_pedestal_feet; collision box size=0.77 0.7 0.31
- link iiwa7_link_0: geometry collision mesh filename=meshes/collision/link_0.stl; visual mesh filename=meshes/visual/link_0.stl
- link iiwa7_link_1: geometry collision mesh filename=meshes/collision/link_1.stl; visual mesh filename=meshes/visual/link_1.stl
- link iiwa7_link_2: geometry collision mesh filename=meshes/collision/link_2.stl; visual mesh filename=meshes/visual/link_2.stl
- link iiwa7_link_3: geometry collision mesh filename=meshes/collision/link_3.stl; visual mesh filename=meshes/visual/link_3.stl
- link iiwa7_link_4: geometry collision mesh filename=meshes/collision/link_4.stl; visual mesh filename=meshes/visual/link_4.stl
- link iiwa7_link_5: geometry collision mesh filename=meshes/collision/link_5.stl; visual mesh filename=meshes/visual/link_5.stl
- link iiwa7_link_6: geometry collision mesh filename=meshes/collision/link_6.stl; visual mesh filename=meshes/visual/link_6.stl
- link iiwa7_link_7: geometry collision mesh filename=meshes/collision/link_7.stl; visual mesh filename=meshes/visual/link_7.stl
Joints:
- removed joint controller_box_fixed
- removed joint pedestal_feet_fixed
- removed joint pedestal_fixed
- added joint iiwa7_controller_box_fixed: type fixed, parent iiwa7_link_0, child iiwa7_controller_box, origin xyz=0.0 0.0 0.0 rpy=0 0 0
- added joint iiwa7_pedestal_feet_fixed: type fixed, parent iiwa7_link_0, child iiwa7_pedestal_feet, origin xyz=0.0 0.0 0.0 rpy=0 0 0
- added joint iiwa7_pedestal_fixed: type fixed, parent iiwa7_link_0, child iiwa7_pedestal, origin xyz=0.0 0.0 0.0 rpy=0 0 0

File: ur5e/ur5e.urdf (robot description, URDF)
Before this commit: robot ur5e, 11 links, 10 joints
Links:
- link ur5e_base_link: geometry collision mesh filename=meshes/collision/base.stl; visual mesh filename=meshes/visual/base_vis.stl
- link ur5e_forearm_link: geometry collision mesh filename=meshes/collision/forearm.stl; visual mesh filename=meshes/visual/forearm_vis.stl
- link ur5e_shoulder_link: geometry collision mesh filename=meshes/collision/shoulder.stl; visual mesh filename=meshes/visual/shoulder_vis.stl
- link ur5e_upper_arm_link: geometry collision mesh filename=meshes/collision/upperarm.stl; visual mesh filename=meshes/visual/upperarm_vis.stl
- link ur5e_ur5e_pedestal: geometry collision cylinder length=0.62 radius=0.18; visual mesh filename=meshes/ur5e_pedestal/pedestal.STL
- link ur5e_wrist_1_link: geometry collision mesh filename=meshes/collision/wrist1.stl; visual mesh filename=meshes/visual/wrist1_vis.stl
- link ur5e_wrist_2_link: geometry collision mesh filename=meshes/collision/wrist2.stl; visual mesh filename=meshes/visual/wrist2_vis.stl
- link ur5e_wrist_3_link: geometry collision mesh filename=meshes/collision/wrist3.stl; visual mesh filename=meshes/visual/wrist3_vis.stl
