Commit message: modified ur5e

File: ur5e/ur5e.urdf (robot description, URDF)
Before this commit: robot ur5e, 11 links, 10 joints
Links:
- removed link base_link
- removed link ee_link
- removed link forearm_link
- removed link shoulder_link
- removed link upper_arm_link
- removed link ur5e_controller_box
- removed link ur5e_pedestal
- removed link ur5e_pedestal_feet
- removed link wrist_1_link
- removed link wrist_2_link
- removed link wrist_3_link
- added link ur5e_base_link, mass 4.0; collision mesh filename=meshes/ur5e/collision/base.stl; visual mesh filename=meshes/ur5e/visual/base_vis.stl
- added link ur5e_forearm_link, mass 2.275; collision mesh filename=meshes/ur5e/collision/forearm.stl; visual mesh filename=meshes/ur5e/visual/forearm_vis.stl
- added link ur5e_right_hand; collision box size=0.01 0.01 0.01
- added link ur5e_shoulder_link, mass 3.7; collision mesh filename=meshes/ur5e/collision/shoulder.stl; visual mesh filename=meshes/ur5e/visual/shoulder_vis.stl
- added link ur5e_upper_arm_link, mass 8.393; collision mesh filename=meshes/ur5e/collision/upperarm.stl; visual mesh filename=meshes/ur5e/visual/upperarm_vis.stl
- added link ur5e_ur5e_controller_box; collision box size=0.22 0.4 0.53
- added link ur5e_ur5e_pedestal, mass 60.86397744; collision cylinder length=0.62 radius=0.18; visual mesh filename=meshes/ur5e/ur5e_pedestal/pedestal.STL
- added link ur5e_ur5e_pedestal_feet; collision box size=0.77 0.7 0.31
- added link ur5e_wrist_1_link, mass 1.219; collision mesh filename=meshes/ur5e/collision/wrist1.stl; visual mesh filename=meshes/ur5e/visual/wrist1_vis.stl
- added link ur5e_wrist_2_link, mass 1.219; collision mesh filename=meshes/ur5e/collision/wrist2.stl; visual mesh filename=meshes/ur5e/visual/wrist2_vis.stl
- added link ur5e_wrist_3_link, mass 0.1879; collision mesh filename=meshes/ur5e/collision/wrist3.stl; visual mesh filename=meshes/ur5e/visual/wrist3_vis.stl
Joints:
- joint ee_fixed_joint: child ee_link -> ur5e_right_hand; origin xyz=0.0 0.0823 0.0 rpy=0.0 0.0 1.570796325 -> xyz=0 0.098 0 rpy=0 0.0 1.5707963; parent wrist_3_link -> ur5e_wrist_3_link
- joint elbow_joint: child forearm_link -> ur5e_forearm_link; origin xyz=0.0 -0.1197 0.425 rpy=0.0 0.0 0.0 -> xyz=0.0 -0.131 0.425 rpy=0.0 0.0 0.0; parent upper_arm_link -> ur5e_upper_arm_link
- joint shoulder_lift_joint: child upper_arm_link -> ur5e_upper_arm_link; origin xyz=0.0 0.13585 0.0 rpy=0.0 1.570796325 0.0 -> xyz=0.0 0.138 0.0 rpy=0.0 1.570796325 0.0; parent shoulder_link -> ur5e_shoulder_link
- joint shoulder_pan_joint: child shoulder_link -> ur5e_shoulder_link; origin xyz=0.0 0.0 0.089159 rpy=0.0 0.0 0.0 -> xyz=0.0 0.0 0.163 rpy=0.0 0.0 0.0; parent base_link -> ur5e_base_link
- joint ur5e_controller_box_fixed: child controller_box -> ur5e_controller_box; parent base -> ur5e_base
- joint ur5e_pedestal_feet_fixed: child base_link -> ur5e_base_link; parent pedestal_feet -> ur5e_pedestal_feet
- joint ur5e_pedestal_fixed: child base_link -> ur5e_base_link; parent ur5e_pedestal -> ur5e_ur5e_pedestal
- joint wrist_1_joint: child wrist_1_link -> ur5e_wrist_1_link; origin xyz=0.0 0.0 0.39225 rpy=0.0 1.570796325 0.0 -> xyz=0 0 0.392 rpy=0.0 1.570796325 0.0; parent forearm_link -> ur5e_forearm_link
- joint wrist_2_joint: child wrist_2_link -> ur5e_wrist_2_link; origin xyz=0.0 0.093 0.0 rpy=0.0 0.0 0.0 -> xyz=0.0 0.127 0.0 rpy=0.0 0.0 0.0; parent wrist_1_link -> ur5e_wrist_1_link
- joint wrist_3_joint: child wrist_3_link -> ur5e_wrist_3_link; origin xyz=0.0 0.0 0.09465 rpy=0.0 0.0 0.0 -> xyz=0 0 0.1 rpy=0.0 0.0 0.0; parent wrist_2_link -> ur5e_wrist_2_link

Commit message: modified ur5e

File: ur5e/ur5e.urdf (robot description, URDF)
Before this commit: robot ur5e, 11 links, 10 joints
Links:
- removed link ur5e_ur5e_controller_box
- removed link ur5e_ur5e_pedestal
- removed link ur5e_ur5e_pedestal_feet
- added link ur5e_controller_box; collision box size=0.22 0.4 0.53
- added link ur5e_pedestal, mass 60.86397744; collision cylinder length=0.62 radius=0.18; visual mesh filename=meshes/ur5e_pedestal/pedestal.STL
- added link ur5e_pedestal_feet; collision box size=0.77 0.7 0.31
Joints:
- joint ur5e_controller_box_fixed: parent ur5e_base -> ur5e_base_link
- joint ur5e_pedestal_feet_fixed: child ur5e_base_link -> ur5e_pedestal_feet; parent ur5e_pedestal_feet -> ur5e_base_link
- joint ur5e_pedestal_fixed: child ur5e_base_link -> ur5e_pedestal; parent ur5e_ur5e_pedestal -> ur5e_base_link
